Commit message: refactor meshes and urdf

File: buzzmobile/simulation/models/buzzmobile/urdf/buzzmobile.urdf (robot description, URDF)
Before this commit: robot buzzmobile, 14 links, 13 joints
Links:
- link chassis: geometry collision mesh filename=package://buzzmobile/simulation/models/buzzmobile/meshes/bu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; visual mesh filename=package://buzzmobile/simulation/models/buzzmobile/meshes/bu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
- link wheel_back_left: geometry collision mesh filename=package://buzzmobile/simulation/models/buzzmobile/mesh/whee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; visual mesh filename=package://buzzmobile/simulation/models/buzzmobile/mesh/whee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
- link wheel_back_right: geometry collision mesh filename=package://buzzmobile/simulation/models/buzzmobile/mesh/whee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; visual mesh filename=package://buzzmobile/simulation/models/buzzmobile/mesh/whee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
- link wheel_front_left: geometry collision mesh filename=package://buzzmobile/simulation/models/buzzmobile/mesh/whee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; visual mesh filename=package://buzzmobile/simulation/models/buzzmobile/mesh/whee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
- link wheel_front_right: geometry collision mesh filename=package://buzzmobile/simulation/models/buzzmobile/mesh/whee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; visual mesh filename=package://buzzmobile/simulation/models/buzzmobile/mesh/whee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

Commit message: it all compiles now! (fixed broke CMake+launchers+urdf)

File: buzzmobile/simulation/models/buzzmobile/urdf/buzzmobile.urdf (robot description, URDF)
Before this commit: robot buzzmobile, 14 links, 13 joints
Links:
- link chassis: geometry collision mesh filename=package://buzzmobile/simulation/models/buzzmobile/mesh/buzz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; visual mesh filename=package://buzzmobile/simulation/models/buzzmobile/mesh/buzz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
