Commit message: update joints with mesh filenames

File: buzzmobile/simulation/models/car/car_joints.urdf (robot description, URDF)
Before this commit: robot buzzmobile, 14 links, 13 joints
Links:
- link chassis: geometry collision mesh filename=package://buzzmobile/simulation/models/car/car_mesh.dae; visual mesh filename=package://buzzmobile/simulation/models/car/car_mesh.dae
- link wheel_back_left: geometry collision mesh filename=package://buzzmobile/simulation/models/car/wheel_mesh.dae; visual mesh filename=package://buzzmobile/simulation/models/car/wheel_mesh.dae
- link wheel_back_right: geometry collision mesh filename=package://buzzmobile/simulation/models/car/wheel_mesh.dae; visual mesh filename=package://buzzmobile/simulation/models/car/wheel_mesh.dae
- link wheel_front_left: geometry collision mesh filename=package://buzzmobile/simulation/models/car/wheel_mesh.dae; visual mesh filename=package://buzzmobile/simulation/models/car/wheel_mesh.dae
- link wheel_front_right: geometry collision mesh filename=package://buzzmobile/simulation/models/car/wheel_mesh.dae; visual mesh filename=package://buzzmobile/simulation/models/car/wheel_mesh.dae

Commit message: added all the gps stuffs

File: buzzmobile/simulation/models/car/car_joints.urdf (robot description, URDF)
Before this commit: robot buzzmobile, 14 links, 13 joints
Links:
- removed link imu
- added link gps
Joints:
- removed joint imu
- added joint gps: type fixed, parent chassis, child gps, origin xyz=0 0 0.1778 rpy=0 0 0

Commit message: it renders!

File: buzzmobile/simulation/models/car/car_joints.urdf (robot description, URDF)
Before this commit: robot buzzmobile, 14 links, 13 joints
Links:
- link back_axle: mass 0.001 -> 3.311
- link chassis: mass 5.0 -> 136.0
- link steering_front_left: mass 0.001 -> 2
- link steering_front_right: mass 0.001 -> 0.1
- link wheel_back_left: mass 0.1 -> 2
- link wheel_back_right: mass 0.1 -> 2
- link wheel_front_left: mass 0.1 -> 2
- link wheel_front_right: mass 0.1 -> 2
Joints:
- joint axle_to_left_wheel: origin xyz=0 0.14439 0 rpy=0 0 0 -> xyz=0 0.645 0 rpy=0 0 0
- joint axle_to_right_wheel: origin xyz=0 -0.14439 0 rpy=0 0 0 -> xyz=0 0 0 rpy=0 0 0
- joint base_footprint_to_chassis: origin xyz=0 0 0.036 rpy=0 0 0 -> xyz=0 0 0.3302 rpy=0 0 0
- joint chassis_to_left_steering: origin xyz=0.33246 0.14366 0 rpy=0 0 0 -> xyz=2.032 0.645 0 rpy=0 0 0
- joint chassis_to_right_steering: origin xyz=0.33246 -0.14366 0 rpy=0 0 0 -> xyz=2.032 -0.645 0 rpy=0 0 0

Commit message: included imu in navsatfix

File: buzzmobile/simulation/models/car/car_joints.urdf (robot description, URDF)
Before this commit: robot buzzmobile, 14 links, 13 joints
Links:
- added link imu

Commit message: the car urdf now has both an imu and a urdf

File: buzzmobile/simulation/models/car/car_joints.urdf (robot description, URDF)
Before this commit: robot buzzmobile, 15 links, 13 joints
Joints:
- added joint imu: type fixed, parent chassis, child imu, origin xyz=0 0 0.1 rpy=0 0 0

Commit message: many changes, makes car move, albeit slowly

File: buzzmobile/simulation/models/car/car_joints.urdf (robot description, URDF)
Before this commit: robot buzzmobile, 14 links, 13 joints
Links:
- link back_axle: mass 3.311 -> 0.001
- link chassis: mass 136.0 -> 5.0
- link steering_front_left: mass 2 -> 0.001
- link steering_front_right: mass 0.1 -> 0.001
- link wheel_back_left: mass 2 -> 0.1
- link wheel_back_right: mass 2 -> 0.1
- link wheel_front_right: mass 2 -> 0.1

Commit message: fixed most mistakes requested on the PR

File: buzzmobile/simulation/models/car/car_joints.urdf (robot description, URDF)
Before this commit: robot buzzmobile, 15 links, 14 joints
Joints:
- joint lidar_joint: origin xyz=0.255 0 5 rpy=0 0 0 -> xyz=2 0 0 rpy=0 0 0

Commit message: more precise URDF and specified in constants.yaml problem with rosparam serv

File: buzzmobile/simulation/models/car/car_joints.urdf (robot description, URDF)
Before this commit: robot buzzmobile, 15 links, 14 joints
Joints:
- joint lidar_joint: origin xyz=2 0 0 rpy=0 0 0 -> xyz=2.182 0 0 rpy=0 0 0
